Commit message: Added 3d camera

File: irobot_create_description/urdf/create3.urdf.xacro (robot description, xacro)
@@ -11,4 +11,9 @@
   <xacro:include filename="$(find irobot_create_description)/urdf/sensors/optical_mouse.urdf.xacro"/>
   <xacro:include filename="$(find irobot_create_description)/urdf/wheel_with_wheeldrop.urdf.xacro" />
+  <xacro:arg name="camera_visual" default="true"/>
+  <xacro:property name="r200_cam_rgb_px" value="0.005"/>
+  <xacro:property name="r200_cam_rgb_py" value="0.018"/>
+  <xacro:property name="r200_cam_rgb_pz" value="0.013"/>
+  <xacro:property name="r200_cam_depth_offset" value="0.01"/>
   <!-- Mechanical properties -->
   <xacro:property name="body_z_offset"           value="${-2.5*cm2m}" />
@@ -199,3 +204,69 @@
     </plugin>
   </gazebo>
+   <link name="camera_link">
+  <visual>
+    <origin xyz="0 0 0" rpy="0 0 0"/>
+    <geometry>
+      <box size="0.012 0.067 0.023"/>
+    </geometry>
+  </visual>
+  <collision>
+    <origin xyz="0 0 0" rpy="0 0 0"/>
+    <geometry>
+      <box size="0.012 0.067 0.023"/>
+    </geometry>
+  </collision>
+  <inertial>
+    <origin xyz="0 0 0" rpy="0 0 0"/>
+    <mass value="0.035"/>
+    <inertia ixx="0.001"  ixy="0"  ixz="0" iyy="0.001" iyz="0" izz="0.001" />
+  </inertial>
+</link>
+<joint name="camera_joint" type="fixed">
+  <parent link="base_link"/>
+  <child link="camera_link"/>
+  <origin xyz="${caster_position_x + 0.01} 0 0.105" rpy="0 0 0"/>
+</joint>
+<link name="camera_depth_frame"/>
+<joint name="camera_depth_joint" type="fixed">
+  <origin xyz="0 0 0" rpy="${-pi/2} 0 ${-pi/2}"/>
+  <parent link="camera_link"/>
+  <child link="camera_depth_frame"/>
+</joint>
+<gazebo reference="camera_link">
+  <sensor name="depth_camera" type="depth">
+    <visualize>true</visualize>
+    <update_rate>30.0</update_rate>
+    <camera name="camera">
+      <horizontal_fov>1.047198</horizontal_fov>
+      <image>
+        <width>640</width>
+        <height>480</height>
+        <format>R8G8B8</format>
+      </image>
+      <clip>
+        <near>0.05</near>
+        <far>3</far>
+      </clip>
+    </camera>
+    <plugin name="depth_camera_controller" filename="libgazebo_ros_camera.so">
+      <baseline>0.2</baseline>
+      <alwaysOn>true</alwaysOn>
+      <updateRate>0.0</updateRate>
+      <frame_name>camera_depth_frame</frame_name>
+      <pointCloudCutoff>0.5</pointCloudCutoff>
+      <pointCloudCutoffMax>3.0</pointCloudCutoffMax>
+      <distortionK1>0</distortionK1>
+      <distortionK2>0</distortionK2>
+      <distortionK3>0</distortionK3>
+      <distortionT1>0</distortionT1>
+      <distortionT2>0</distortionT2>
+      <CxPrime>0</CxPrime>
+      <Cx>0</Cx>
+      <Cy>0</Cy>
+      <focalLength>0</focalLength>
+      <hackBaseline>0</hackBaseline>
+    </plugin>
+  </sensor>
+</gazebo>
 </robot>

Commit message: added arm base and 3d camera

File: irobot_create_description/urdf/create3.urdf.xacro (robot description, xacro)
@@ -204,5 +204,30 @@
     </plugin>
   </gazebo>
-   <link name="camera_link">
+<!-- Arm base definition-->
+<link name="arm_base_link">
+  <visual>
+    <origin xyz="-0.06 0 0.096" rpy="0 0 0"/>
+    <geometry>
+      <mesh filename="file://$(find irobot_create_description)/meshes/arm/base.stl" scale="0.001 0.001 0.001"/>
+    </geometry>
+  </visual>
+  <!-- <collision>
+    <origin xyz="0 0 0" rpy="0 0 0"/>
+    <geometry>
+      <box size="0.012 0.067 0.023"/>
+    </geometry>
+  </collision> -->
+  <!-- <inertial>
+    <origin xyz="0 0 0" rpy="0 0 0"/>
+    <mass value="0.035"/>
+    <inertia ixx="0.001"  ixy="0"  ixz="0" iyy="0.001" iyz="0" izz="0.001" />
+  </inertial> -->
+</link>
+<joint name="arm_base_joint" type="fixed">
+  <parent link="base_link"/>
+  <child link="arm_base_link"/>
+</joint>
+  <!-- Camera -->
+<link name="camera_link">
   <visual>
     <origin xyz="0 0 0" rpy="0 0 0"/>

Commit message: added arm and camera to independent urdf files usign fixed joints

File: irobot_create_description/urdf/create3.urdf.xacro (robot description, xacro)
@@ -8,7 +8,9 @@
   <xacro:include filename="$(find irobot_create_description)/urdf/sensors/imu.urdf.xacro" />
   <xacro:include filename="$(find irobot_create_description)/urdf/sensors/ir_intensity.urdf.xacro" />
+  <xacro:include filename="$(find irobot_create_description)/urdf/sensors/rgbd_camera.urdf.xacro" />
   <xacro:include filename="$(find irobot_create_description)/urdf/sensors/ir_opcode_receivers.urdf.xacro" />
   <xacro:include filename="$(find irobot_create_description)/urdf/sensors/optical_mouse.urdf.xacro"/>
   <xacro:include filename="$(find irobot_create_description)/urdf/wheel_with_wheeldrop.urdf.xacro" />
+  <xacro:include filename="$(find irobot_create_description)/urdf/arm.urdf.xacro" />
   <xacro:arg name="camera_visual" default="true"/>
   <xacro:property name="r200_cam_rgb_px" value="0.005"/>
@@ -154,4 +156,10 @@
     <origin xyz="0.0399 0.1488 ${ir_intensity_z_pos + base_link_z_offset}" rpy="0 0 1.309"/>
   </xacro:ir_intensity>
+  <xacro:rgbd_camera name="camera">
+    <origin xyz="0.14 0 ${0.045 + base_link_z_offset}" rpy="0 0 0"/>
+  </xacro:rgbd_camera>
+  <xacro:hephestus_arm>
+      <origin xyz="-0.06 0 0.096" rpy="0 0 0"/>
+  </xacro:hephestus_arm>
   <!-- Buttons -->
   <xacro:button
@@ -204,94 +212,3 @@
     </plugin>
   </gazebo>
-<!-- Arm base definition-->
-<link name="arm_base_link">
-  <visual>
-    <origin xyz="-0.06 0 0.096" rpy="0 0 0"/>
-    <geometry>
-      <mesh filename="file://$(find irobot_create_description)/meshes/arm/base.stl" scale="0.001 0.001 0.001"/>
-    </geometry>
-  </visual>
-  <!-- <collision>
-    <origin xyz="0 0 0" rpy="0 0 0"/>
-    <geometry>
-      <box size="0.012 0.067 0.023"/>
-    </geometry>
-  </collision> -->
-  <!-- <inertial>
-    <origin xyz="0 0 0" rpy="0 0 0"/>
-    <mass value="0.035"/>
-    <inertia ixx="0.001"  ixy="0"  ixz="0" iyy="0.001" iyz="0" izz="0.001" />
-  </inertial> -->
-</link>
-<joint name="arm_base_joint" type="fixed">
-  <parent link="base_link"/>
-  <child link="arm_base_link"/>
-</joint>
-  <!-- Camera -->
-<link name="camera_link">
-  <visual>
-    <origin xyz="0 0 0" rpy="0 0 0"/>
-    <geometry>
-      <box size="0.012 0.067 0.023"/>
-    </geometry>
-  </visual>
-  <collision>
-    <origin xyz="0 0 0" rpy="0 0 0"/>
-    <geometry>
-      <box size="0.012 0.067 0.023"/>
-    </geometry>
-  </collision>
-  <inertial>
-    <origin xyz="0 0 0" rpy="0 0 0"/>
-    <mass value="0.035"/>
-    <inertia ixx="0.001"  ixy="0"  ixz="0" iyy="0.001" iyz="0" izz="0.001" />
-  </inertial>
-</link>
-<joint name="camera_joint" type="fixed">
-  <parent link="base_link"/>
-  <child link="camera_link"/>
-  <origin xyz="${caster_position_x + 0.01} 0 0.105" rpy="0 0 0"/>
-</joint>
-<link name="camera_depth_frame"/>
-<joint name="camera_depth_joint" type="fixed">
-  <origin xyz="0 0 0" rpy="${-pi/2} 0 ${-pi/2}"/>
-  <parent link="camera_link"/>
-  <child link="camera_depth_frame"/>
-</joint>
-<gazebo reference="camera_link">
-  <sensor name="depth_camera" type="depth">
-    <visualize>true</visualize>
-    <update_rate>30.0</update_rate>
-    <camera name="camera">
-      <horizontal_fov>1.047198</horizontal_fov>
-      <image>
-        <width>640</width>
-        <height>480</height>
-        <format>R8G8B8</format>
-      </image>
-      <clip>
-        <near>0.05</near>
-        <far>3</far>
-      </clip>
-    </camera>
-    <plugin name="depth_camera_controller" filename="libgazebo_ros_camera.so">
-      <baseline>0.2</baseline>
-      <alwaysOn>true</alwaysOn>
-      <updateRate>0.0</updateRate>
-      <frame_name>camera_depth_frame</frame_name>
-      <pointCloudCutoff>0.5</pointCloudCutoff>
-      <pointCloudCutoffMax>3.0</pointCloudCutoffMax>
-      <distortionK1>0</distortionK1>
-      <distortionK2>0</distortionK2>
-      <distortionK3>0</distortionK3>
-      <distortionT1>0</distortionT1>
-      <distortionT2>0</distortionT2>
-      <CxPrime>0</CxPrime>
-      <Cx>0</Cx>
-      <Cy>0</Cy>
-      <focalLength>0</focalLength>
-      <hackBaseline>0</hackBaseline>
-    </plugin>
-  </sensor>
-</gazebo>
 </robot>

File: irobot_create_description/urdf/sensors/rgbd_camera.urdf.xacro (robot description, xacro)
@@ -1,26 +1,71 @@
 <?xml version="1.0"?>
 <robot xmlns:xacro="http://ros.org/wiki/xacro">
-  <xacro:macro name="optical_mouse" params="name:=mouse parent_link:=base_link update_rate:=62 *origin" >
+<xacro:macro name="rgbd_camera" params="name:=camera parent_link:=base_link update_rate:=60 *origin">
     <joint name="${name}_joint" type="fixed">
-      <xacro:insert_block name="origin"/>
-      <parent link="${parent_link}"/>
-      <child link="${name}"/>
-    </joint>
-    <link name="${name}">
-      <xacro:inertial_dummy />
-    </link>
-    <gazebo>
-      <plugin name="${name}_plugin" filename="libgazebo_ros_create_optical_mouse.so">
-          <ros>
-            <namespace>/</namespace>
-            <remapping>~/out:=${name}</remapping>
-          </ros>
-        <update_rate>${update_rate}</update_rate>
-        <link_name>${name}</link_name>
+    <xacro:insert_block name="origin"/>
+    <parent link="${parent_link}"/>
+    <child link="${name}_link"/>
+  </joint>
+  <link name="${name}_link">
+    <visual>
+      <origin xyz="0 0 0" rpy="0 0 0"/>
+      <geometry>
+        <box size="0.012 0.067 0.023"/>
+      </geometry>
+    </visual>
+    <collision>
+      <origin xyz="0 0 0" rpy="0 0 0"/>
+      <geometry>
+        <box size="0.012 0.067 0.023"/>
+      </geometry>
+    </collision>
+    <inertial>
+      <origin xyz="0 0 0" rpy="0 0 0"/>
+      <mass value="0.035"/>
+      <inertia ixx="0"  ixy="0"  ixz="0" iyy="0" iyz="0" izz="0" />
+    </inertial>
+  </link>
+  <link name="${name}_depth_frame"/>
+  <joint name="${name}_depth_joint" type="fixed">
+    <origin xyz="0 0 0" rpy="${-pi/2} 0 ${-pi/2}"/>
+    <parent link="${name}_link"/>
+    <child link="${name}_depth_frame"/>
+  </joint>
+  <gazebo reference="${name}_link">
+    <sensor name="depth_camera" type="depth">
+      <visualize>true</visualize>
+      <update_rate>${update_rate}</update_rate>
+      <camera name="camera">
+        <horizontal_fov>1.047198</horizontal_fov>
+        <image>
+          <width>640</width>
+          <height>480</height>
+          <format>R8G8B8</format>
+        </image>
+        <clip>
+          <near>0.05</near>
+          <far>3</far>
+        </clip>
+      </camera>
+      <plugin name="depth_camera_controller" filename="libgazebo_ros_camera.so">
+        <baseline>0.2</baseline>
+        <alwaysOn>true</alwaysOn>
+        <updateRate>0.0</updateRate>
+        <frame_name>camera_depth_frame</frame_name>
+        <pointCloudCutoff>0.5</pointCloudCutoff>
+        <pointCloudCutoffMax>3.0</pointCloudCutoffMax>
+        <distortionK1>0</distortionK1>
+        <distortionK2>0</distortionK2>
+        <distortionK3>0</distortionK3>
+        <distortionT1>0</distortionT1>
+        <distortionT2>0</distortionT2>
+        <CxPrime>0</CxPrime>
+        <Cx>0</Cx>
+        <Cy>0</Cy>
+        <focalLength>0</focalLength>
+        <hackBaseline>0</hackBaseline>
       </plugin>
-    </gazebo>
-    <gazebo reference="${name}_joint" >
-      <preserveFixedJoint>true</preserveFixedJoint>
-    </gazebo>
-  </xacro:macro>
+    </sensor>
+  </gazebo>
+</xacro:macro>
 </robot>
