Commit message: robot arm in rviz, working on joint fixes

File: irobot_create_description/urdf/arm.urdf.xacro (robot description, xacro)
@@ -2,4 +2,22 @@
 <robot xmlns:xacro="http://ros.org/wiki/xacro">
 <xacro:macro name="hephestus_arm" params="name:=arm parent_link:=base_link *origin">
+  <!-- Transmission macro -->
+  <xacro:macro name="SimpleTransmission" params="joint n motor">
+    <transmission name="tran${n}">
+      <type>transmission_interface/SimpleTransmission</type>
+      <joint name="${joint}">
+        <hardwareInterface>hardware_interface/PositionJointInterface</hardwareInterface>
+      </joint>
+      <actuator name="${motor}">
+        <hardwareInterface>hardware_interface/PositionJointInterface</hardwareInterface>
+        <mechanicalReduction>1</mechanicalReduction>
+      </actuator>
+    </transmission>
+  </xacro:macro>
+    <xacro:macro name="box_inertia" params="m x y z">
+            <inertia  ixx="${m*(y*y+z*z)/12}" ixy = "0" ixz = "0"
+                    iyy="${m*(x*x+z*z)/12}" iyz = "0"
+                    izz="${m*(x*x+z*z)/12}" />
+    </xacro:macro>
   <!-- Arm base definition-->
     <link name="${name}_base_link">
@@ -29,9 +47,9 @@
             </geometry>
         </visual>
-        <!-- <inertial>
-            <origin xyz="0 0 0" rpy="0 0 0"/>
-            <mass value="0.063"/>
-            <inertia ixx="0"  ixy="0"  ixz="0" iyy="0" iyz="0" izz="0" />
-       </inertial> -->
+    <inertial>
+        <origin xyz="0 0 0" rpy="0 0 0"/>
+        <mass value="0.065"/>
+        <xacro:box_inertia m="0.063" x="0.020" y="0.040" z="0.04"/>
+    </inertial>
     </link>
     <xacro:property name="link_1_angle" value="-1.57"/>
@@ -49,17 +67,17 @@
             </geometry>
         </visual>
-        <!-- <inertial>
-            <origin xyz="0 0 0" rpy="0 0 0"/>
-            <mass value="0.093"/>
-            <inertia ixx="0"  ixy="0"  ixz="0" iyy="0" iyz="0" izz="0" />
-       </inertial> -->
-    </link>
-    <joint name="${name}_link1_joint" type="fixed">
-        <!-- <limit effort="1000.0" lower="-3.14" upper="3.14" velocity="0.5"/> -->
-           <axis xyz="0 0 1"/>
+        <inertial>
+			<mass value="2e-06"/>
+			<inertia ixx="1.1e-09" ixy="0" ixz="0" iyy="1.1e-09" iyz="0" izz="1.1e-09"/>
+		</inertial>
+    </link>
+    <joint name="${name}_link1_joint" type="revolute">
+        <limit effort="1000.0" lower="-3.14" upper="3.14" velocity="0.5"/>
+        <axis xyz="0 0 1"/>
         <parent link="${name}_motor_1_link"/>
         <child link="${name}_link1_link"/>
         <origin xyz="0 0 0" rpy="0 0 ${link_1_angle}"/>
     </joint>
+    <xacro:SimpleTransmission n="1" joint="${name}_link1_joint" motor="${name}_motor_1_link" />
     <!-- motor 2 definition-->
     <link name="${name}_motor_2_link">
@@ -72,7 +90,7 @@
         <inertial>
             <origin xyz="0 0 0" rpy="0 0 0"/>
-            <mass value="0.063"/>
-            <inertia ixx="0"  ixy="0"  ixz="0" iyy="0" iyz="0" izz="0" />
-       </inertial>
+            <mass value="0.065"/>
+            <xacro:box_inertia m="0.063" x="0.020" y="0.040" z="0.04"/>
+        </inertial>
     </link>
     <joint name="${name}_motor_2_joint" type="fixed">
@@ -127,9 +145,9 @@
             </geometry>
         </visual>
-        <!-- <inertial>
-            <origin xyz="0 0 0" rpy="0 0 0"/>
-            <mass value="0.063"/>
-            <inertia ixx="0"  ixy="0"  ixz="0" iyy="0" iyz="0" izz="0" />
-       </inertial> -->
+        <inertial>
+        <origin xyz="0 0 0" rpy="0 0 0"/>
+        <mass value="0.065"/>
+        <xacro:box_inertia m="0.063" x="0.020" y="0.040" z="0.04"/>
+    </inertial>
     </link>
     <joint name="motor_3_joint" type="fixed">
@@ -184,9 +202,9 @@
         </geometry>
     </visual>
-    <!-- <inertial>
-        <origin xyz="0 0 0" rpy="0 0 0"/>
-        <mass value="0.063"/>
-        <inertia ixx="0"  ixy="0"  ixz="0" iyy="0" iyz="0" izz="0" />
-   </inertial> -->
+    <inertial>
+        <origin xyz="0 0 0" rpy="0 0 0"/>
+        <mass value="0.065"/>
+        <xacro:box_inertia m="0.063" x="0.020" y="0.040" z="0.04"/>
+    </inertial>
     </link>
     <joint name="motor_4_joint" type="fixed">
@@ -222,9 +240,9 @@
             </geometry>
         </visual>
-        <!-- <inertial>
-            <origin xyz="0 0 0" rpy="0 0 0"/>
-            <mass value="0.063"/>
-            <inertia ixx="0"  ixy="0"  ixz="0" iyy="0" iyz="0" izz="0" />
-       </inertial> -->
+        <inertial>
+        <origin xyz="0 0 0" rpy="0 0 0"/>
+        <mass value="0.065"/>
+        <xacro:box_inertia m="0.063" x="0.020" y="0.040" z="0.04"/>
+    </inertial>
     </link>
     <joint name="motor_5_joint" type="fixed">
@@ -279,9 +297,9 @@
             </geometry>
         </visual>
-        <!-- <inertial>
-            <origin xyz="0 0 0" rpy="0 0 0"/>
-            <mass value="0.063"/>
-            <inertia ixx="0"  ixy="0"  ixz="0" iyy="0" iyz="0" izz="0" />
-       </inertial> -->
+        <inertial>
+        <origin xyz="0 0 0" rpy="0 0 0"/>
+        <mass value="0.065"/>
+        <xacro:box_inertia m="0.063" x="0.020" y="0.040" z="0.04"/>
+    </inertial>
     </link>
     <joint name="motor_6_joint" type="fixed">
